Commit message: Checkpoint 1 - Task 1

File: my_rb1_description/urdf/my_rb1_robot.urdf (robot description, URDF)
Before this commit: robot my_rb1_robot, 7 links, 6 joints
Links:
- link back_caster: mass 1 -> ${caster_mass}; geometry collision sphere radius=${caster_radius}; collision sphere radius=0.05
- link base_link: mass 25 -> ${cylinder_mass}; geometry collision cylinder length=${cylinder_height} radius=${cylinder_radius}; visual cylinder length=${cylinder_height} radius=${cylinder_radius}
- link front_caster: mass 1 -> ${caster_mass}; geometry collision sphere radius=${caster_radius}; collision sphere radius=0.05
- link left_wheel: mass 1 -> ${wheel_mass}; geometry collision cylinder length=${wheel_height} radius=${wheel_radius}; visual cylinder length=${wheel_height} radius=${wheel_radius}
- link right_wheel: mass 1 -> ${wheel_mass}; geometry collision cylinder length=${wheel_height} radius=${wheel_radius}; visual cylinder length=${wheel_height} radius=${wheel_radius}
Joints:
- joint joint_laser: origin xyz=0.25 0 0.075 rpy=3.14159265359 0 0 -> xyz=0.25 0 0.075 rpy=${M_PI} 0 0
